File: AmpV2.sch (KiCad schematic (older format))
At the start: 1 part

Commit message: making layout
Parts:
- removed U?: TPA3126D2, Package_SO:HTSSOP-32-1EP_6.1x11mm_P0.65mm_EP5.2x11mm_Mask4.11x4.36mm, symbol CustomLibrary:TPA3126D2
- added C37, C38, C39, C41, C42: CP_Small, Capacitor_SMD:C_0603_1608Metric_Pad1.08x0.95mm_HandSolder, symbol Device:CP_Small
- added C40, C43, C44, C45: C_Small, Capacitor_SMD:C_0603_1608Metric_Pad1.08x0.95mm_HandSolder, symbol Device:C_Small
- added J2: Conn_01x04, Connector_JST:JST_PH_S4B-PH-K_1x04_P2.00mm_Horizontal, symbol Connector_Generic:Conn_01x04
- added J5, J6: OSTTC022162, digikey-footprints:Term_Block_1x2_P5.08MM, symbol dk_Terminal-Blocks-Wire-to-Board:OSTTC022162
- added Q6: BC107, Package_TO_SOT_THT:TO-18-3, symbol Transistor_BJT:BC107
- added R23, R24, R25, R26, R27, R28, R29, R30, R31, R32: R_Small, Resistor_SMD:R_0603_1608Metric_Pad0.98x0.95mm_HandSolder, symbol Device:R_Small
- added S1, S2: EG1218, digikey-footprints:Switch_Slide_11.6x4mm_EG1218, symbol dk_Slide-Switches:EG1218
- added U6: TDA7265, Package_TO_SOT_THT:TO-220-11_P3.4x5.08mm_StaggerOdd_Lead4.85mm_Vertical, symbol CustomLibrary:TDA7265
- added Z1: 1N5231BTR, digikey-footprints:DO-35, symbol dk_Diodes-Zener-Single:1N5231BTR
Connections:
- new net: C40.1, C41.2, U6.1 (-V), U6.6 (-V)
- new net: R29.2, R30.1, U6.10 (IN-(1))
- new net: C39.1, U6.11 (IN+(1))
- new net: J2.4 (Pin_4), J5.1, R29.1, R32.1, U6.2 (OUTPUT(1))
- new net: J2.1 (Pin_1), J6.1, R27.1, R31.1, U6.4 (OUTPUT(2))
- new net: C37.2, Q6.3 (C), R24.2, U6.5 (MUTE)
- new net: C38.1, U6.7 (IN+(2))
- new net: R27.2, R28.1, U6.8 (IN-(2))
- new net: Q6.1 (E), R25.1, R26.1
- new net: Q6.2 (B), R23.1, Z1.K
- new net: R25.2, S2.2
- new net: R23.2, S1.2
- new net: C44.1, R31.2
- new net: C45.1, R32.2
- new net GND: C40.2, C41.1, C42.2, C43.2, C44.2, C45.2, J2.2 (Pin_2), J2.3 (Pin_3), J5.2, J6.2, R26.2, R28.2, R30.2, S1.3, S2.3, U6.9 (GND), Z1.A
- new net VS: C37.1, C42.1, C43.1, R24.1, S1.1, U6.3 (+V)
- no-connect marks 0 -> 1

Commit message: before downsizing
Parts:
- J5: value OSTTC022162 -> OSTTC022162 (R)
- J6: value OSTTC022162 -> OSTTC022162 (L)
Connections:
- net GND: now also J5.1, J6.1; no longer J5.2, J6.2
- net at J2.4 (Pin_4), R29.1, R32.1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: now also J5.2; no longer J5.1
- net at J2.1 (Pin_1), R27.1, R31.1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: now also J6.2; no longer J6.1
- net RIGHTIN: now reaches C39.2
- net LEFTIN: now reaches C38.2
- net VS renamed VIN
Other:
- moved on the sheet: J5
Changed lines of the file:
@@
 	5250 1800 4925 1800
 Wire Wire Line
-	4725 1800 4600 1800
-Wire Wire Line
 	5250 2250 4925 2250
-Wire Wire Line
-	4725 2250 4600 2250
 Wire Wire Line
 	5250 1650 4500 1650
@@
 Wire Wire Line
 	5750 975  5750 1350
-Wire Wire Line
-	5750 975  5750 875
 Connection ~ 5750 975
-$Comp
-L power:VS #PWR0205
-U 1 1 61B74BFC
-P 5750 875
-F 0 "#PWR0205" H 5550 725 50  0001 C CNN
-F 1 "VS" H 5765 1048 50  0000 C CNN
-F 2 "" H 5750 875 50  0001 C CNN
-F 3 "" H 5750 875 50  0001 C CNN
-	1    5750 875
-	1    0    0    -1
-$EndComp
 $Comp
 L Device:C_Small C43
@@
 L dk_Terminal-Blocks-Wire-to-Board:OSTTC022162 J6
 U 1 1 61C2CB5E
-P 9025 1475
-F 0 "J6" V 9024 1297 50  0000 R CNN
-F 1 "OSTTC022162" V 9115 1297 50  0000 R CNN
-F 2 "digikey-footprints:Term_Block_1x2_P5.08MM" H 9225 1675 60  0001 L CNN
-F 3 "http://www.on-shore.com/wp-content/uploads/OSTTCXX2162.pdf" H 9225 1775 60  0001 L CNN
-F 4 "ED2609-ND" H 9225 1875 60  0001 L CNN "Digi-Key_PN"
-F 5 "OSTTC022162" H 9225 1975 60  0001 L CNN "MPN"
-F 6 "Connectors, Interconnects" H 9225 2075 60  0001 L CNN "Category"
-F 7 "Terminal Blocks - Wire to Board" H 9225 2175 60  0001 L CNN "Family"
-F 8 "http://www.on-shore.com/wp-content/uploads/OSTTCXX2162.pdf" H 9225 2275 60  0001 L CNN "DK_Datasheet_Link"
-F 9 "/product-detail/en/on-shore-technology-inc/OSTTC022162/ED2609-ND/614558" H 9225 2375 60  0001 L CNN "DK_Detail_Page"
-F 10 "TERM BLK 2P SIDE ENT 5.08MM PCB" H 9225 2475 60  0001 L CNN "Description"
-F 11 "On Shore Technology Inc." H 9225 2575 60  0001 L CNN "Manufacturer"
-F 12 "Active" H 9225 2675 60  0001 L CNN "Status"
-	1    9025 1475
-	0    -1   1    0
+P 9025 1575
+F 0 "J6" V 9024 1397 50  0000 R CNN
+F 1 "OSTTC022162 (L)" V 9115 1397 50  0000 R CNN
+F 2 "digikey-footprints:Term_Block_1x2_P5.08MM" H 9225 1775 60  0001 L CNN
+F 3 "http://www.on-shore.com/wp-content/uploads/OSTTCXX2162.pdf" H 9225 1875 60  0001 L CNN
+F 4 "ED2609-ND" H 9225 1975 60  0001 L CNN "Digi-Key_PN"
+F 5 "OSTTC022162" H 9225 2075 60  0001 L CNN "MPN"
+F 6 "Connectors, Interconnects" H 9225 2175 60  0001 L CNN "Category"
+F 7 "Terminal Blocks - Wire to Board" H 9225 2275 60  0001 L CNN "Family"
+F 8 "http://www.on-shore.com/wp-content/uploads/OSTTCXX2162.pdf" H 9225 2375 60  0001 L CNN "DK_Datasheet_Link"
+F 9 "/product-detail/en/on-shore-technology-inc/OSTTC022162/ED2609-ND/614558" H 9225 2475 60  0001 L CNN "DK_Detail_Page"
+F 10 "TERM BLK 2P SIDE ENT 5.08MM PCB" H 9225 2575 60  0001 L CNN "Description"
+F 11 "On Shore Technology Inc." H 9225 2675 60  0001 L CNN "Manufacturer"
+F 12 "Active" H 9225 2775 60  0001 L CNN "Status"
+	1    9025 1575
+	0    -1   -1   0
 $EndComp
 $Comp
 L dk_Terminal-Blocks-Wire-to-Board:OSTTC022162 J5
 U 1 1 61C35EF8
-P 9000 2150
-F 0 "J5" V 9091 1972 50  0000 R CNN
-F 1 "OSTTC022162" V 9000 1972 50  0000 R CNN
-F 2 "digikey-footprints:Term_Block_1x2_P5.08MM" H 9200 2350 60  0001 L CNN
-F 3 "http://www.on-shore.com/wp-content/uploads/OSTTCXX2162.pdf" H 9200 2450 60  0001 L CNN
-F 4 "ED2609-ND" H 9200 2550 60  0001 L CNN "Digi-Key_PN"
-F 5 "OSTTC022162" H 9200 2650 60  0001 L CNN "MPN"
-F 6 "Connectors, Interconnects" H 9200 2750 60  0001 L CNN "Category"
-F 7 "Terminal Blocks - Wire to Board" H 9200 2850 60  0001 L CNN "Family"
-F 8 "http://www.on-shore.com/wp-content/uploads/OSTTCXX2162.pdf" H 9200 2950 60  0001 L CNN "DK_Datasheet_Link"
-F 9 "/product-detail/en/on-shore-technology-inc/OSTTC022162/ED2609-ND/614558" H 9200 3050 60  0001 L CNN "DK_Detail_Page"
-F 10 "TERM BLK 2P SIDE ENT 5.08MM PCB" H 9200 3150 60  0001 L CNN "Description"
-F 11 "On Shore Technology Inc." H 9200 3250 60  0001 L CNN "Manufacturer"
-F 12 "Active" H 9200 3350 60  0001 L CNN "Status"
-	1    9000 2150
+P 9025 2250
+F 0 "J5" V 9116 2072 50  0000 R CNN
+F 1 "OSTTC022162 (R)" V 9025 2072 50  0000 R CNN
+F 2 "digikey-footprints:Term_Block_1x2_P5.08MM" H 9225 2450 60  0001 L CNN
+F 3 "http://www.on-shore.com/wp-content/uploads/OSTTCXX2162.pdf" H 9225 2550 60  0001 L CNN
+F 4 "ED2609-ND" H 9225 2650 60  0001 L CNN "Digi-Key_PN"
+F 5 "OSTTC022162" H 9225 2750 60  0001 L CNN "MPN"
+F 6 "Connectors, Interconnects" H 9225 2850 60  0001 L CNN "Category"
+F 7 "Terminal Blocks - Wire to Board" H 9225 2950 60  0001 L CNN "Family"
+F 8 "http://www.on-shore.com/wp-content/uploads/OSTTCXX2162.pdf" H 9225 3050 60  0001 L CNN "DK_Datasheet_Link"
+F 9 "/product-detail/en/on-shore-technology-inc/OSTTC022162/ED2609-ND/614558" H 9225 3150 60  0001 L CNN "DK_Detail_Page"
+F 10 "TERM BLK 2P SIDE ENT 5.08MM PCB" H 9225 3250 60  0001 L CNN "Description"
+F 11 "On Shore Technology Inc." H 9225 3350 60  0001 L CNN "Manufacturer"
+F 12 "Active" H 9225 3450 60  0001 L CNN "Status"
+	1    9025 2250
 	0    -1   -1   0
 $EndComp
@@
 $EndComp
 Wire Wire Line
-	8775 1750 8775 1725
-Wire Wire Line
 	8775 1575 8925 1575
-Wire Wire Line
-	8900 2050 8900 1725
-Wire Wire Line
-	8900 1725 8775 1725
-Connection ~ 8775 1725
-Wire Wire Line
-	8775 1725 8775 1575
-Wire Wire Line
-	7975 2150 8900 2150
 Connection ~ 7975 2150
 Wire Wire Line
@@
 	1    0    0    -1
 $EndComp
+Text Label 4475 1800 0    50   ~ 0
+LEFTIN
+Wire Wire Line
+	4475 1800 4725 1800
+Text Label 4475 2250 0    50   ~ 0
+RIGHTIN
+Wire Wire Line
+	4475 2250 4725 2250
+Wire Wire Line
+	5750 750  5975 750
+Wire Wire Line
+	5750 750  5750 975
+Text Label 5825 750  0    50   ~ 0
+VIN
+Wire Wire Line
+	8775 1575 8775 1750
+Wire Wire Line
+	7975 2150 8925 2150
+$Comp
+L power:GND #PWR0119
+U 1 1 61BF2190
+P 8775 2425
+F 0 "#PWR0119" H 8775 2175 50  0001 C CNN
+F 1 "GND" H 8780 2252 50  0000 C CNN
+F 2 "" H 8775 2425 50  0001 C CNN
+F 3 "" H 8775 2425 50  0001 C CNN
+	1    8775 2425
+	1    0    0    -1
+$EndComp
+Wire Wire Line
+	8925 2250 8775 2250
+Wire Wire Line
+	8775 2250 8775 2425
 $EndSCHEMATC

Commit message: gonna try auto-route
Parts:
- S1, S2: footprint digikey-footprints:Switch_Slide_11.6x4mm_EG1218 -> digikey-footprints:Switch_Slide_JS202011SCQN
Connections:
- net LEFTIN renamed LINEIN_L
- net RIGHTIN renamed LINEIN_R
Other:
- moved on the sheet: R25, R26, S2
Changed lines of the file:
@@
 L Device:R_Small R25
 U 1 1 61B8359A
-P 4075 2400
-F 0 "R25" H 4134 2446 50  0000 L CNN
-F 1 "R_Small" H 4134 2355 50  0000 L CNN
-F 2 "Resistor_SMD:R_0603_1608Metric_Pad0.98x0.95mm_HandSolder" H 4075 2400 50  0001 C CNN
-F 3 "~" H 4075 2400 50  0001 C CNN
-	1    4075 2400
+P 4075 2575
+F 0 "R25" H 4134 2621 50  0000 L CNN
+F 1 "R_Small" H 4134 2530 50  0000 L CNN
+F 2 "Resistor_SMD:R_0603_1608Metric_Pad0.98x0.95mm_HandSolder" H 4075 2575 50  0001 C CNN
+F 3 "~" H 4075 2575 50  0001 C CNN
+	1    4075 2575
 	1    0    0    -1
 $EndComp
@@
 L Device:R_Small R26
 U 1 1 61B84059
-P 4325 2400
-F 0 "R26" H 4384 2446 50  0000 L CNN
-F 1 "R_Small" H 4384 2355 50  0000 L CNN
-F 2 "Resistor_SMD:R_0603_1608Metric_Pad0.98x0.95mm_HandSolder" H 4325 2400 50  0001 C CNN
-F 3 "~" H 4325 2400 50  0001 C CNN
-	1    4325 2400
+P 4325 2575
+F 0 "R26" H 4384 2621 50  0000 L CNN
+F 1 "R_Small" H 4384 2530 50  0000 L CNN
+F 2 "Resistor_SMD:R_0603_1608Metric_Pad0.98x0.95mm_HandSolder" H 4325 2575 50  0001 C CNN
+F 3 "~" H 4325 2575 50  0001 C CNN
+	1    4325 2575
 	1    0    0    -1
 $EndComp
@@
 L power:GND #PWR0208
 U 1 1 61B8464A
-P 4325 2600
-F 0 "#PWR0208" H 4325 2350 50  0001 C CNN
-F 1 "GND" H 4330 2427 50  0000 C CNN
-F 2 "" H 4325 2600 50  0001 C CNN
-F 3 "" H 4325 2600 50  0001 C CNN
-	1    4325 2600
+P 4325 2775
+F 0 "#PWR0208" H 4325 2525 50  0001 C CNN
+F 1 "GND" H 4330 2602 50  0000 C CNN
+F 2 "" H 4325 2775 50  0001 C CNN
+F 3 "" H 4325 2775 50  0001 C CNN
+	1    4325 2775
 	1    0    0    -1
 $EndComp
@@
 L power:GND #PWR0209
 U 1 1 61B847E0
-P 4175 3150
-F 0 "#PWR0209" H 4175 2900 50  0001 C CNN
-F 1 "GND" H 4180 2977 50  0000 C CNN
-F 2 "" H 4175 3150 50  0001 C CNN
-F 3 "" H 4175 3150 50  0001 C CNN
-	1    4175 3150
+P 4175 3325
+F 0 "#PWR0209" H 4175 3075 50  0001 C CNN
+F 1 "GND" H 4180 3152 50  0000 C CNN
+F 2 "" H 4175 3325 50  0001 C CNN
+F 3 "" H 4175 3325 50  0001 C CNN
+	1    4175 3325
 	-1   0    0    -1
 $EndComp
 Wire Wire Line
-	4075 2100 4075 2225
-Wire Wire Line
-	4325 2500 4325 2600
+	4325 2675 4325 2775
 Wire Wire Line
 	3775 1900 3725 1900
 Wire Wire Line
 	3725 1900 3725 2025
-$Comp
-L power:GND #PWR0210
-U 1 1 61B8CE5F
-P 3725 2525
-F 0 "#PWR0210" H 3725 2275 50  0001 C CNN
-F 1 "GND" H 3730 2352 50  0000 C CNN
-F 2 "" H 3725 2525 50  0001 C CNN
-F 3 "" H 3725 2525 50  0001 C CNN
-	1    3725 2525
-	1    0    0    -1
-$EndComp
 Wire Wire Line
 	3725 2425 3725 2525
@@
 F 0 "S1" H 3175 1575 50  0000 C CNN
 F 1 "EG1218" H 3175 1666 50  0000 C CNN
-F 2 "digikey-footprints:Switch_Slide_11.6x4mm_EG1218" H 3375 2100 50  0001 L CNN
+F 2 "digikey-footprints:Switch_Slide_JS202011SCQN" H 3375 2100 50  0001 L CNN
 F 3 "http://spec_sheets.e-switch.com/specs/P040040.pdf" H 3375 2200 60  0001 L CNN
 F 4 "EG1903-ND" H 3375 2300 60  0001 L CNN "Digi-Key_PN"
@@
 Wire Wire Line
 	2975 2000 2975 2350
-$Comp
-L dk_Slide-Switches:EG1218 S2
-U 1 1 61BA12E5
-P 4075 2825
-F 0 "S2" V 4029 2969 50  0000 L CNN
-F 1 "EG1218" V 4120 2969 50  0000 L CNN
-F 2 "digikey-footprints:Switch_Slide_11.6x4mm_EG1218" H 4275 3025 50  0001 L CNN
-F 3 "http://spec_sheets.e-switch.com/specs/P040040.pdf" H 4275 3125 60  0001 L CNN
-F 4 "EG1903-ND" H 4275 3225 60  0001 L CNN "Digi-Key_PN"
-F 5 "EG1218" H 4275 3325 60  0001 L CNN "MPN"
-F 6 "Switches" H 4275 3425 60  0001 L CNN "Category"
-F 7 "Slide Switches" H 4275 3525 60  0001 L CNN "Family"
-F 8 "http://spec_sheets.e-switch.com/specs/P040040.pdf" H 4275 3625 60  0001 L CNN "DK_Datasheet_Link"
-F 9 "/product-detail/en/e-switch/EG1218/EG1903-ND/101726" H 4275 3725 60  0001 L CNN "DK_Detail_Page"
-F 10 "SWITCH SLIDE SPDT 200MA 30V" H 4275 3825 60  0001 L CNN "Description"
-F 11 "E-Switch" H 4275 3925 60  0001 L CNN "Manufacturer"
-F 12 "Active" H 4275 4025 60  0001 L CNN "Status"
-	1    4075 2825
-	0    -1   1    0
-$EndComp
-Wire Wire Line
-	4175 3150 4175 3025
-NoConn ~ 3975 3025
-Wire Wire Line
-	4075 2225 4325 2225
-Wire Wire Line
-	4325 2225 4325 2300
-Connection ~ 4075 2225
-Wire Wire Line
-	4075 2225 4075 2300
-Wire Wire Line
-	4075 2625 4075 2500
+Wire Wire Line
+	4175 3325 4175 3200
+NoConn ~ 3975 3200
+Wire Wire Line
+	4075 2400 4325 2400
+Wire Wire Line
+	4325 2400 4325 2475
+Connection ~ 4075 2400
+Wire Wire Line
+	4075 2400 4075 2475
+Wire Wire Line
+	4075 2800 4075 2675
 $Comp
 L dk_Diodes-Zener-Single:1N5231BTR Z1
@@
 P 3725 2225
 F 0 "Z1" V 3778 2147 60  0000 R CNN
-F 1 "1N5231BTR" V 3672 2147 60  0000 R CNN
+F 1 "1N5231BTR" V 3600 2475 60  0000 R CNN
 F 2 "digikey-footprints:DO-35" H 3925 2425 60  0001 L CNN
 F 3 "https://www.onsemi.com/pub/Collateral/1N5221B-D.PDF" H 3925 2525 60  0001 L CNN
@@
 	1    0    0    -1
 $EndComp
-Text Label 4475 1800 0    50   ~ 0
-LEFTIN
-Wire Wire Line
-	4475 1800 4725 1800
-Text Label 4475 2250 0    50   ~ 0
-RIGHTIN
-Wire Wire Line
-	4475 2250 4725 2250
 Wire Wire Line
 	5750 750  5975 750
@@
 Wire Wire Line
 	8775 2250 8775 2425
+$Comp
+L dk_Slide-Switches:EG1218 S2
+U 1 1 61BA12E5
+P 4075 3000
+F 0 "S2" V 4029 3144 50  0000 L CNN
+F 1 "EG1218" V 4120 3144 50  0000 L CNN
+F 2 "digikey-footprints:Switch_Slide_JS202011SCQN" H 4275 3200 50  0001 L CNN
+F 3 "http://spec_sheets.e-switch.com/specs/P040040.pdf" H 4275 3300 60  0001 L CNN
+F 4 "EG1903-ND" H 4275 3400 60  0001 L CNN "Digi-Key_PN"
+F 5 "EG1218" H 4275 3500 60  0001 L CNN "MPN"
+F 6 "Switches" H 4275 3600 60  0001 L CNN "Category"
+F 7 "Slide Switches" H 4275 3700 60  0001 L CNN "Family"
+F 8 "http://spec_sheets.e-switch.com/specs/P040040.pdf" H 4275 3800 60  0001 L CNN "DK_Datasheet_Link"
+F 9 "/product-detail/en/e-switch/EG1218/EG1903-ND/101726" H 4275 3900 60  0001 L CNN "DK_Detail_Page"
+F 10 "SWITCH SLIDE SPDT 200MA 30V" H 4275 4000 60  0001 L CNN "Description"
+F 11 "E-Switch" H 4275 4100 60  0001 L CNN "Manufacturer"
+F 12 "Active" H 4275 4200 60  0001 L CNN "Status"
+	1    4075 3000
+	0    -1   1    0
+$EndComp
+$Comp
+L power:GND #PWR0210
+U 1 1 61B8CE5F
+P 3725 2525
+F 0 "#PWR0210" H 3725 2275 50  0001 C CNN
+F 1 "GND" H 3730 2352 50  0000 C CNN
+F 2 "" H 3725 2525 50  0001 C CNN
+F 3 "" H 3725 2525 50  0001 C CNN
+	1    3725 2525
+	1    0    0    -1
+$EndComp
+Text HLabel 4600 1800 0    50   Input ~ 0
+LINEIN_L
+Wire Wire Line
+	4600 1800 4725 1800
+Text HLabel 4600 2250 0    50   Input ~ 0
+LINEIN_R
+Wire Wire Line
+	4600 2250 4725 2250
+Wire Wire Line
+	4075 2100 4075 2400
+Text HLabel 5975 750  2    50   Input ~ 0
+VIN
 $EndSCHEMATC
