File: TeensyAudioShield.sch (KiCad schematic (older format))
At the start: 26 parts, among them CON2 Headphone, CON3 Line In, U5 SGTL5000XNAA3

Commit message: gonna try auto-route
Connections:
- net GNDA is gone; now on net GND: C34.2, RV2.3, U5.7 (AGND)
- net D15-A1-RX3-SPDIF_IN renamed CTRL_ADR0_CS
- net D18-A4-SDA0 renamed CTRL_DATA
- net D19-A5-SCL0 renamed CTRL_CLK
- net D20-A6-TX5-LRCLK1 renamed I2S_LRCLK
- net D21-A7-RX5-BCLK1 renamed I2S_SCLK
- net D23-A9-CRX1-MCLK1 renamed SYS_MCLK
- net D7-RX2-OUT1A renamed I2S_DIN
- net D8-TX2-IN1 renamed I2S_DOUT
- net LEFTIN renamed LINEOUT_L
- net RIGHTIN renamed LINEOUT_R
